File: kicad/mss-debug/mss-debug.kicad_sch (KiCad schematic)
At the start: 79 parts, among them Q1 Si2333, SW1 JS202011SCQN, U1 AP3012, U2 AP3012

Commit message: Initial cut of the 2.0 board
Parts:
- removed D?: GREEN LED, LED_SMD:LED_0805_2012Metric, symbol Device:LED
- removed H1, H2, H3, H4: MountingHole, MountingHole:MountingHole_3.2mm_M3_Pad, symbol Mechanical:MountingHole_Pad
- removed R?: 1k, Resistor_SMD:R_0805_2012Metric, symbol Device:R_US
- added C11: 22uF, Capacitor_SMD:C_0805_2012Metric, symbol Device:C
- added D3: GREEN LED, LED_SMD:LED_0805_2012Metric, symbol Device:LED
- added R4: 1k, Resistor_SMD:R_0805_2012Metric, symbol Device:R_US
- added unit 4 of U3
- added unit 5 of U4
- added unit 6 of U4
- added unit 4 of U4
- added unit 3 of U4
- BT1: footprint (none) -> Battery:BatteryHolder_Keystone_2479_3xAAA
- Q1: footprint (none) -> Package_TO_SOT_SMD:SOT-23
- R16: renamed from R?; value 10k -> 1k
- R18, R20, R27, R29, R31: renamed from R?; value 10k -> 1K
- SW1: footprint (none) -> ISE_UltraLibrarian:SW_JS202011SCQN
- SW2, SW3, SW4, SW5, SW6, SW7, SW8: renamed from SW?; footprint (none) -> ISE_UltraLibrarian:SW_JS202011SCQN
- gave numbers to parts that had none: 46
Connections:
- net GND: now also R18.2, R20.2, R27.2, R29.2, R31.2, C11.2, R4.1, U3.9, U4.11, U4.14, U4.7, U4.9; no longer D5.1 (K), D6.1 (K), D7.1 (K), D8.1 (K), D9.1 (K)
- net at R27.1: now also D7.1 (K); no longer D7.2 (A)
- net at SW5.3 (C): now also SW5.6 (C)
- net at L1.1, L2.1, Q1.2 (S)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: now also C11.1, D3.2 (A)
- net at R18.1: now also D5.1 (K); no longer D5.2 (A)
- net at R29.1: now also D8.1 (K); no longer D8.2 (A)
- net at C6.1, R17.1: now also U3.14; no longer U3.3
- net at U3.2: now also D9.2 (A); no longer R31.2
- net at C8.1, R26.1: now also U3.7; no longer U3.3
- net at R31.1: now also D9.1 (K); no longer D9.2 (A)
- net at C5.1, R11.1: now also U4.5; no longer U4.3
- net at C9.1, R28.1: now also U3.5; no longer U3.3
- net at SW2.1 (A), U4.3: now also U4.4; no longer U4.2
- net at SW7.3 (C): now also SW7.6 (C)
- net at C7.1, R19.1: now also U3.11; no longer U3.3
- net at SW4.3 (C): now also SW4.6 (C)
- net at R20.1: now also D6.1 (K); no longer D6.2 (A)
- net at SW6.3 (C): now also SW6.6 (C)
- new net: D7.2 (A), U3.6
- new net: D5.2 (A), U3.15
- new net: D6.2 (A), U3.12
- new net: D3.1 (K), R4.2
- new net: D8.2 (A), U3.4
Other:
- moved on the sheet: BT1, C2, C3, D5, D6, D7, D8, D9, Q1, R18, R20, R27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
